File: Dial_Tone_Generator.sch (KiCad schematic (older format))
At the start: 46 parts, among them J1 AUDIO_OUT, J2 DC_IN, U1 LMC6484, U2 LM317L_TO92

Commit message: some schematic changes
Connections:
- net GND: now also RV3.2
- net at C9.1, D2.2 (A), R18.2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: no longer RV3.2
Changed lines of the file:
@@
 	8250 5210 8250 5100
 Wire Wire Line
-	7720 5930 7960 5930
-Wire Wire Line
-	7960 5930 7960 5600
-Connection ~ 7960 5600
-Wire Wire Line
-	7960 5600 7570 5600
+	7720 5930 7880 5930
 $Comp
 L power:GND #PWR0103
@@
 $EndComp
 Connection ~ 8250 5600
-Wire Wire Line
-	7960 5600 8250 5600
 $Comp
 L power:GND #PWR0117
@@
 	1    0    0    -1
 $EndComp
+Wire Wire Line
+	7570 5600 8250 5600
+Wire Wire Line
+	7880 5930 7880 6080
+$Comp
+L power:GND #PWR?
+U 1 1 6408C7C3
+P 7880 6080
+F 0 "#PWR?" H 7880 5830 50  0001 C CNN
+F 1 "GND" H 7885 5907 50  0000 C CNN
+F 2 "" H 7880 6080 50  0001 C CNN
+F 3 "" H 7880 6080 50  0001 C CNN
+	1    7880 6080
+	1    0    0    -1
+$EndComp
