File: Dial_Tone_Generator.kicad_pcb (KiCad board)
At the start: 2 copper layers, 88.9 x 63.5 mm, 0 parts

Commit message: Some PCB cleanup
Parts:
- added C1: 0.1uF, Capacitor_THT:C_Rect_L10.3mm_W5.7mm_P7.50mm_MKS4, F.Cu at (149.4, 113.3)
- added C10: 1000uF, Capacitor_THT:CP_Radial_D14.0mm_P5.00mm, F.Cu at (122.2, 83.8)
- added C2: 0.1uF, Capacitor_THT:C_Rect_L10.3mm_W5.7mm_P7.50mm_MKS4, F.Cu at (168.7, 113.3)
- added C3: 1uF, Capacitor_THT:CP_Radial_D5.0mm_P2.50mm, F.Cu at (160.0, 103.1)
- added C4: 470pF, Capacitor_THT:C_Disc_D5.1mm_W3.2mm_P5.00mm, F.Cu at (137.9, 78.5)
- added C5: 0.1uF, Capacitor_THT:C_Rect_L10.3mm_W5.7mm_P7.50mm_MKS4, F.Cu at (156.2, 80.0)
- added C6: 0.1uF, Capacitor_THT:C_Rect_L10.3mm_W5.7mm_P7.50mm_MKS4, F.Cu at (170.9, 80.0)
- added C7: 4700pF, Capacitor_THT:C_Disc_D5.1mm_W3.2mm_P5.00mm, F.Cu at (165.1, 78.5)
- added C8: 1uF, Capacitor_THT:CP_Radial_D5.0mm_P2.50mm, F.Cu at (176.5, 84.8)
- added C9: 10uF, Capacitor_THT:CP_Radial_D5.0mm_P2.50mm, F.Cu at (112.0, 113.0)
- added D1: 1N4002, Diode_THT:D_DO-41_SOD81_P10.16mm_Horizontal, F.Cu at (118.1, 75.9)
- added D2: 1N4002, Diode_THT:D_DO-41_SOD81_P10.16mm_Horizontal, F.Cu at (118.9, 99.6)
- added D3: 1N4002, Diode_THT:D_DO-41_SOD81_P10.16mm_Horizontal, F.Cu at (122.2, 96.0)
- added H1: MountingHole, MountingHole:MountingHole_3.2mm_M3, F.Cu at (105.4, 67.3)
- added H2: MountingHole, MountingHole:MountingHole_3.2mm_M3, F.Cu at (186.7, 67.3)
- added H3: MountingHole, MountingHole:MountingHole_3.2mm_M3, F.Cu at (186.7, 123.2)
- added H4: MountingHole, MountingHole:MountingHole_3.2mm_M3, F.Cu at (105.4, 123.2)
- added J1: AUDIO_OUT, TerminalBlock:TerminalBlock_bornier-2_P5.08mm, F.Cu at (184.2, 97.8)
- added J2: DC_IN, TerminalBlock:TerminalBlock_bornier-2_P5.08mm, F.Cu at (108.0, 81.8)
- added R1: 30.1K, Resistor_THT:R_Axial_DIN0207_L6.3mm_D2.5mm_P10.16mm_Horizontal, F.Cu at (157.5, 122.2)
- added R10: 470K, Resistor_THT:R_Axial_DIN0207_L6.3mm_D2.5mm_P10.16mm_Horizontal, F.Cu at (173.5, 92.7)
- added R11: 1M, Resistor_THT:R_Axial_DIN0207_L6.3mm_D2.5mm_P10.16mm_Horizontal, F.Cu at (141.5, 81.0)
- added R12: 470K, Resistor_THT:R_Axial_DIN0207_L6.3mm_D2.5mm_P10.16mm_Horizontal, F.Cu at (150.6, 70.9)
- added R13: 470K, Resistor_THT:R_Axial_DIN0207_L6.3mm_D2.5mm_P10.16mm_Horizontal, F.Cu at (147.6, 81.0)
- added R14: 56K, Resistor_THT:R_Axial_DIN0207_L6.3mm_D2.5mm_P10.16mm_Horizontal, F.Cu at (144.5, 70.9)
- added R15: 10K, Resistor_THT:R_Axial_DIN0207_L6.3mm_D2.5mm_P10.16mm_Horizontal, F.Cu at (161.5, 81.0)
- added R16: 470R, Resistor_THT:R_Axial_DIN0207_L6.3mm_D2.5mm_P10.16mm_Horizontal, F.Cu at (176.5, 81.0)
- added R17: 470K, Resistor_THT:R_Axial_DIN0207_L6.3mm_D2.5mm_P10.16mm_Horizontal, F.Cu at (176.5, 92.7)
- added R18: 240R, Resistor_THT:R_Axial_DIN0207_L6.3mm_D2.5mm_P10.16mm_Horizontal, F.Cu at (115.6, 99.6)
- added R2: 30.1K, Resistor_THT:R_Axial_DIN0207_L6.3mm_D2.5mm_P10.16mm_Horizontal, F.Cu at (154.4, 112.0)
- added R3: 178K, Resistor_THT:R_Axial_DIN0207_L6.3mm_D2.5mm_P10.16mm_Horizontal, F.Cu at (144.3, 112.0)
- added R4: 78.7K, Resistor_THT:R_Axial_DIN0207_L6.3mm_D2.5mm_P10.16mm_Horizontal, F.Cu at (141.2, 112.0)
- added R5: 1M, Resistor_THT:R_Axial_DIN0207_L6.3mm_D2.5mm_P10.16mm_Horizontal, F.Cu at (143.8, 92.7)
- added R6: 30.1K, Resistor_THT:R_Axial_DIN0207_L6.3mm_D2.5mm_P10.16mm_Horizontal, F.Cu at (160.5, 122.2)
- added R7: 30.1K, Resistor_THT:R_Axial_DIN0207_L6.3mm_D2.5mm_P10.16mm_Horizontal, F.Cu at (163.6, 112.0)
- added R8: 178K, Resistor_THT:R_Axial_DIN0207_L6.3mm_D2.5mm_P10.16mm_Horizontal, F.Cu at (173.7, 112.0)
- added R9: 61.9K, Resistor_THT:R_Axial_DIN0207_L6.3mm_D2.5mm_P10.16mm_Horizontal, F.Cu at (176.8, 112.0)
- added RV1: 10K, Potentiometer_THT:Potentiometer_Bourns_3299Y_Vertical, F.Cu at (136.9, 116.8)
- added RV2: 10K, Potentiometer_THT:Potentiometer_Bourns_3299Y_Vertical, F.Cu at (183.4, 116.8)
- added RV3: 5K, Potentiometer_THT:Potentiometer_Bourns_3299Y_Vertical, F.Cu at (118.9, 115.1)
- added TP1: 350TP, TestPoint:TestPoint_Loop_D2.50mm_Drill1.0mm, F.Cu at (144.3, 108.7)
- added TP2: 440TP, TestPoint:TestPoint_Loop_D2.50mm_Drill1.0mm, F.Cu at (173.7, 108.7)
- added TP3: +7.5V, TestPoint:TestPoint_Loop_D2.50mm_Drill1.0mm, F.Cu at (127.5, 102.9)
- added TP4: GND, TestPoint:TestPoint_Loop_D2.50mm_Drill1.0mm, F.Cu at (137.7, 102.9)
- added U1: LMC6484, Package_DIP:DIP-14_W7.62mm_LongPads, F.Cu at (152.4, 99.1)
- added U2: LM317L_TO92, Package_TO_SOT_THT:TO-92_Inline_Wide, F.Cu at (109.2, 102.1)
Routing:
- net +7.5V: track 0.00 -> 176.1 mm
- net Net-(C4-Pad2): track 0.00 -> 67.6 mm
- net Net-(C2-Pad1): track 0.00 -> 48.6 mm
- net Net-(C1-Pad1): track 0.00 -> 48.3 mm
- net Net-(R6-Pad2): track 0.00 -> 36.6 mm
- net Net-(R1-Pad2): track 0.00 -> 35.7 mm
- net Net-(C10-Pad1): track 0.00 -> 35.1 mm
- net Net-(C6-Pad2): track 0.00 -> 32.9 mm
- net Net-(C6-Pad1): track 0.00 -> 26.8 mm
- net Net-(C9-Pad1): track 0.00 -> 25.5 mm
- net Net-(C4-Pad1): track 0.00 -> 24.8 mm
- net Net-(C5-Pad1): track 0.00 -> 21.0 mm
- net Net-(R3-Pad1): track 0.00 -> 20.1 mm
- net Net-(R8-Pad1): track 0.00 -> 18.5 mm
- net Net-(C8-Pad2): track 0.00 -> 17.3 mm
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- added copper zone on F.Cu, net GND
Other:
- net class Default: clearance 0.2 -> 0.2032; trace_width 0.25 -> 0.762; via_dia 0.8 -> 1.524; via_drill 0.4 -> 0.762
- rule trace_clearance: 0.2 -> 0.2032

Commit message: generated gerber files
Parts:
- moved C4 2.03 mm to (135.9, 78.5)
- moved R11 1.78 mm to (139.7, 81.0)
- moved R14 1.78 mm to (142.7, 70.9)
- moved C7 0.25 mm to (165.4, 78.5)
Routing:
- net Net-(C6-Pad2): track 32.9 -> 35.3 mm
- net Net-(C4-Pad1): track 24.8 -> 26.9 mm
- net Net-(C4-Pad2): track 67.6 -> 69.3 mm
Other:
- board text added: "+ -"
- board text added: "+7.5V"
- board text added: "12-24V DC IN"
- board text added: "350HZ ADJ."
- board text added: "350TP"
- board text added: "440HZ ADJ."
- board text added: "440TP"
- board text added: "A G"
- board text added: "AUDIO OUT"
- board text added: "DIAL TONE GENERATOR REV. A"
- board text added: "DMA '23"
- board text added: "GND"
- board text added: "V+ ADJ."
